Commit message: update(code):add pkg robot*

File: src/robot_description/urdf/robot.urdf (robot description, URDF)
Before this commit: robot robot_agv, 7 links, 6 joints
Links:
- link base_link: geometry visual box size=0.52 0.55 0.08
Joints:
- joint base_Bleft_wheel_joint: origin xyz=0.15 -0.16 0.025 rpy=0 0 0 -> xyz=-0.275 -0.260 0.025 rpy=1.5708 0 0
- joint base_Bright_wheel_joint: origin xyz=0.15 0.16 0.025 rpy=0 0 0 -> xyz=-0.275 0.260 0.025 rpy=1.5708 0 0
- joint base_Fleft_wheel_joint: origin xyz=-0.15 -0.16 0.025 rpy=0 0 0 -> xyz=0.275 0.260 0.025 rpy=1.5708 0 0
- joint base_Fright_wheel_joint: axis 0 1 0 -> 0 -1 0; origin xyz=-0.15 0.16 0.025 rpy=0 0 0 -> xyz=0.275 -0.260 0.025 rpy=1.5708 0 0
- joint base_laser_joint: origin xyz=0 0 0.105 rpy=0 0 0 -> xyz=0 -0.02 0.105 rpy=0 0 3.1415
